Commit message: 修改关节角度范围

File: fabo_arm7_gazebo/urdf/fabo_arm7_hokuyo_kinect_2.urdf.xacro (robot description, xacro)
@@ -37,5 +37,5 @@
 	<xacro:property name="arm_angleset_y" value="0.0" />
 	<joint name="bottom_joint" type="fixed">
-		<origin xyz="0.0 -0.20 0.62" rpy="1.57 0 0" />
+		<origin xyz="0.0 -0.10 0.62" rpy="1.57 0 0" />
 		<!-- <origin xyz="${arm_offset_x} ${arm_offset_y} ${arm_offset_z}" rpy="${arm_angleset_r} ${arm_angleset_p} ${arm_angleset_y}"/> -->
 		<parent link="base_footprint"/>
@@ -537,7 +537,8 @@
 		</plugin>
 	</gazebo>
-	<!-- kinectdk -->
+	<!-- kinectdk -->  <!-- ${-M_PI/2} -->
+  	<xacro:property name="M_PI" value="3.1415926535897931" />
 	<xacro:include filename="$(find fabo_arm7_gazebo)/urdf/kinectdk.urdf.xacro"/>
-	<xacro:sensor_kinectdk parent="Link7"/>
+	<xacro:sensor_kinectdk parent="Link7"  cam_oy="${-M_PI/2}"   dis_py_between_rgb_and_depth="0.0"/>
 	<!-- hokuyo -->
     <xacro:include filename="$(find fabo_arm7_gazebo)/urdf/hokuyo.urdf.xacro" />

File: fabo_arm7_gazebo/urdf/fabo_arm7_hokuyo_kinect_fix.urdf.xacro (robot description, xacro)
@@ -22,4 +22,10 @@
 		</inertial>
 	</xacro:macro>
+	<link name="dummy">
+	</link>
+	<joint name="dummy_joint" type="fixed">
+		<parent link="dummy" />
+		<child link="base_footprint" />
+	</joint>
 	<link name="base_footprint">
 		<visual>
@@ -547,5 +553,4 @@
 	</gazebo>
 	<!-- kinectdk -->
-	<xacro:property name="M_PI" value="3.1415926535897931" />
 	<xacro:include filename="$(find fabo_arm7_gazebo)/urdf/kinectdk.urdf.xacro"/>
 	<xacro:sensor_kinectdk parent="Link7"/>

File: fabo_arm7_gazebo/urdf/fabo_arm7_hokuyo_kinect_fix_2.urdf.xacro (robot description, xacro)
@@ -2,7 +2,6 @@
 <robot name="fabo_arm7" xmlns:xacro="http://www.ros.org/wiki/xacro">
 <!-- body -->
-	<xacro:include filename="$(find fabo_arm7_gazebo)/urdf/fabo_body.urdf.xacro" />
-	<!-- Body of mrobot, with plates, standoffs -->
-	<fabo_body/>
+	<!-- <xacro:include filename="$(find fabo_arm7_gazebo)/urdf/fabo_body.urdf.xacro" /> -->
+	<!-- <fabo_body/> -->
 <!-- arm -->
 	<xacro:include filename="$(find rm_75_description)/urdf/rm_75.transmission.xacro"/>
@@ -23,23 +22,32 @@
 		</inertial>
 	</xacro:macro>
-	<!-- <link name="dummy">
-	</link> -->
-	<!-- <joint name="dummy_joint" type="fixed">
+	<link name="dummy">
+	</link>
+	<joint name="dummy_joint" type="fixed">
 		<parent link="dummy" />
 		<child link="base_link_arm" />
-	</joint> -->
+	</joint>
 	<!-- ///////////////////////////////////////   bottom_joint   ////////////////////////////////////////// -->
-	<xacro:property name="arm_offset_x" value="0.0" />
-	<xacro:property name="arm_offset_y" value="-0.20" />
-	<xacro:property name="arm_offset_z" value="0.62" />
-	<xacro:property name="arm_angleset_r" value="1.57" />
-	<xacro:property name="arm_angleset_p" value="0.0" />
-	<xacro:property name="arm_angleset_y" value="0.0" />
 	<joint name="bottom_joint" type="fixed">
-		<origin xyz="0.0 -0.20 0.62" rpy="1.57 0 0" />
-		<!-- <origin xyz="${arm_offset_x} ${arm_offset_y} ${arm_offset_z}" rpy="${arm_angleset_r} ${arm_angleset_p} ${arm_angleset_y}"/> -->
-		<parent link="base_footprint"/>
-		<child link="base_link_arm"/>
-	</joint>
+		<origin xyz="0.0 0 -0.62" rpy="0 0 0" />
+		<parent link="base_link_arm"/>
+		<child link="bottom_link"/>
+	</joint>
+	<link name="bottom_link">
+		<visual>
+		<origin xyz=" 0 0 -0.02"  rpy="0 0 0"/>
+		<geometry>
+			<box size="1 1 0.02" />
+		</geometry>
+		<material name="Brown" />
+		</visual>
+		<collision>
+		<origin xyz=" 0 0 -0.02"  rpy="0 0 0"/>
+		<geometry>
+			<box size="1 1 0.02" />
+		</geometry>
+		</collision>
+		<xacro:Box_inertial_matrix m="500" l="1" w="1" h="0.02"/>
+	</link>
 	<link
 		name="base_link_arm">
@@ -540,9 +548,3 @@
 	<xacro:include filename="$(find fabo_arm7_gazebo)/urdf/kinectdk.urdf.xacro"/>
 	<xacro:sensor_kinectdk parent="Link7"/>
-	<!-- hokuyo -->
-    <xacro:include filename="$(find fabo_arm7_gazebo)/urdf/hokuyo.urdf.xacro" />
-	<xacro:property name="laser_offset_x" value="0.25" />
-	<xacro:property name="laser_offset_y" value="0" />
-	<xacro:property name="laser_offset_z" value="0.1" />
-	<xacro:laser_hokuyo parent="plate_2_link" laser_offset_x="${laser_offset_x}" laser_offset_y="${laser_offset_y}" laser_offset_z="${laser_offset_z}" />
 </robot>

File: fabo_arm7_gazebo/urdf/kinectdk.urdf.xacro (robot description, xacro)
@@ -1,4 +1,5 @@
 <?xml version="1.0"?>
 <robot name="sensor_kinect" xmlns:xacro="http://ros.org/wiki/xacro">
+  <xacro:property name="M_PI" value="3.1415926535897931" />
   <!-- [1]  Microsoft Kinect / ASUS Xtion PRO Live for simulation -->
   <xacro:macro name="sim_3dsensor">
@@ -42,34 +43,25 @@
   </xacro:macro>
   <!-- [2]  pose from camera to robot -->
-  <xacro:property name="cam_px" value="0.0185" />    <!-- 62.5-44=18.5mm  -->
-  <xacro:property name="kinect_cam_py" value="0.0"/>
+  <xacro:property name="cam_px" value="0.004925" />    <!-- 4.925mm  -->
+  <xacro:property name="cam_py" value="0.0"/>
 	<xacro:property name="cam_pz" value="0.02" />
 	<xacro:property name="cam_or" value="0" />
 	<xacro:property name="cam_op" value="0" />
-	<xacro:property name="cam_oy" value="0" />
+	<!-- <xacro:property name="cam_oy" value="${-M_PI/2}" /> -->
+  <!-- <xacro:property name="dis_py_between_rgb_and_depth" value="0.0"/> -->
   <!-- [3]  Parameterised in part by the values in turtlebot_properties.urdf.xacro -->
-  <xacro:macro name="sensor_kinectdk" params="parent">
-    <joint name="camera_rgb_joint" type="fixed">
-      <origin xyz="${cam_px} ${kinect_cam_py} ${cam_pz}" rpy="${cam_or} ${cam_op} ${cam_oy}"/>
+  <xacro:macro name="sensor_kinectdk" params="parent cam_oy dis_py_between_rgb_and_depth ">
+    <!-- joint connected to robot -->
+    <joint name="camera_link_joint" type="fixed">
+      <origin xyz="${cam_px} ${cam_py} ${cam_pz}" rpy="${cam_or} ${cam_op} ${cam_oy}"/>
       <parent link="${parent}"/>
-      <child link="camera_rgb_frame" />
-    </joint>
-    <link name="camera_rgb_frame"/>
-    <joint name="camera_rgb_optical_joint" type="fixed">
-      <origin xyz="0 0 0" rpy="${-M_PI/2} 0 ${-M_PI/2}" />
-      <parent link="camera_rgb_frame" />
-      <child link="camera_rgb_optical_frame" />
-    </joint>
-    <link name="camera_rgb_optical_frame"/>
-    <joint name="camera_joint" type="fixed">
-      <origin xyz="0 ${-kinect_cam_py} 0" rpy="0 0 0"/>
-      <parent link="camera_rgb_frame"/>
       <child link="camera_link"/>
     </joint>
+    <!-- camera body -->
     <link name="camera_link">
       <visual>
-       <origin xyz="0 0 0" rpy="0 0 ${M_PI/2}"/>
+       <origin xyz="0 0 0" rpy="0 0 0"/>
         <geometry>
-          <box size="0.1 0.125 0.04"/>
+          <box size="0.0994 0.1 0.04"/>
         </geometry>
       </visual>
@@ -77,5 +69,5 @@
         <origin xyz="0.0 0.0 0.0" rpy="0 0 0"/>
   	    <geometry>
-  	      <box size="0.1 0.125 0.02"/>
+  	      <box size="0.0994 0.1 0.02"/>
   	    </geometry>
   	  </collision>
@@ -88,9 +80,51 @@
       </inertial>
     </link>
+    <joint name="head_joint" type="fixed">
+      <origin xyz="0.0627 0 0" rpy="0 0 0"/>  <!-- 62.7mm -->
+      <parent link="camera_link"/>
+      <child link="head_link"/>
+    </joint>
+    <link name="head_link">
+      <visual>
+        <origin xyz="0 0 0" rpy="0 0 0"/>
+        <geometry>
+          <box size="0.026 0.105 0.04"/>
+        </geometry>
+      </visual>
+      <collision>
+        <origin xyz="0.0 0.0 0.0" rpy="0 0 0"/>
+        <geometry>
+          <box size="0.026 0.105 0.04"/>
+        </geometry>
+      </collision>
+      <inertial>
+        <mass value="1e-5" /> <!-- 0.564 -->
+        <origin xyz="0 0 0" />
+        <inertia ixx="0.003881243" ixy="0.0" ixz="0.0"
+                  iyy="0.000498940" iyz="0.0"
+                  izz="0.003879257" />
+      </inertial>
+    </link>
+    <gazebo reference="head_link">
+              <material>Gazebo/Red</material>
+    </gazebo>
+    <!-- camera image  -->
+    <joint name="camera_rgb_joint" type="fixed">
+      <origin xyz="0.080625 ${dis_py_between_rgb_and_depth/2} 0" rpy="0 0 0"/>  <!-- 80.625mm -->
+      <parent link="camera_link"/>
+      <child link="camera_rgb_frame" />
+    </joint>
+    <link name="camera_rgb_frame"/>
+    <joint name="camera_rgb_optical_joint" type="fixed">
+      <origin xyz="0 0 0" rpy="${-M_PI/2} 0 ${-M_PI/2}" />
+      <parent link="camera_rgb_frame" />
+      <child link="camera_rgb_optical_frame" />
+    </joint>
+    <link name="camera_rgb_optical_frame"/>
     <!-- The fixed joints & links below are usually published by static_transformers launched by the OpenNi launch
          files. However, for Gazebo simulation we need them, so we add them here.
          (Hence, don't publish them additionally!) -->
 	<joint name="camera_depth_joint" type="fixed">
-	  <origin xyz="0 ${2 * -kinect_cam_py} 0" rpy="0 0 0" />
+	  <origin xyz="0 ${-dis_py_between_rgb_and_depth} 0" rpy="0 0 0" />
 	  <parent link="camera_rgb_frame" />
 	  <child link="camera_depth_frame" />

File: rm_75_description/urdf/rm_75_bottom_zhjd.urdf.xacro (robot description, xacro)
@@ -20,13 +20,8 @@
   <link name="dummy">
   </link>
+  <!-- ///////////////////////////////////////   bottom_joint   ////////////////////////////////////////// -->
   <joint name="dummy_joint" type="fixed">
     <parent link="dummy" />
-    <child link="base_link" />
-  </joint>
-  <!-- ///////////////////////////////////////   bottom_joint   ////////////////////////////////////////// -->
-  <joint name="bottom_joint" type="fixed">
-    <origin xyz="0 0 0" rpy="0 0 0" />
-    <parent link="base_link"/>
-    <child link="bottom_link"/>
+    <child link="bottom_link" />
   </joint>
   <link name="bottom_link">
@@ -34,5 +29,5 @@
       <origin xyz=" 0 0 -0.02"  rpy="0 0 0"/>
       <geometry>
-        <!-- <box size="1 1 0.02" /> -->
+        <box size="1 1 0.02" />
       </geometry>
       <material name="Brown" />
@@ -46,6 +41,34 @@
     <xacro:Box_inertial_matrix m="500" l="1" w="1" h="0.02"/>
   </link>
-  <link
-    name="base_link">
+  <!-- ///////////////////////////////////////   bottom_2_joint   ////////////////////////////////////////// -->
+  <joint name="bottom_2_joint" type="fixed">
+    <origin xyz="0 0 0.4" rpy="0  0 -1.57" />
+    <parent link="bottom_link"/>
+    <child link="bottom_2_link"/>
+  </joint>
+  <link name="bottom_2_link">
+    <visual>
+      <origin xyz=" 0 0 0"  rpy="0 0 0"/>
+      <geometry>
+        <box size="0.5 0.5 0.8" />
+      </geometry>
+      <material name="Brown" />
+    </visual>
+    <collision>
+      <origin xyz=" 0 0 -0.02"  rpy="0 0 0"/>
+      <geometry>
+        <box size="0.5 0.5 0.8" />
+      </geometry>
+    </collision>
+    <xacro:Box_inertial_matrix m="500" l="1" w="1" h="0.02"/>
+  </link>
+  <!-- ///////////////////////////////////////   arm   ////////////////////////////////////////// -->
+  <joint name="base_link_joint" type="fixed">
+    <origin xyz="0.25 0  0.0" rpy="0 1.57 0" />
+    <parent link="bottom_2_link"/>
+    <child link="base_link_arm"/>
+  </joint>
+  <link
+    name="base_link_arm">
     <inertial>
       <origin
@@ -133,5 +156,5 @@
       rpy="-1.5708 0 0" />
     <parent
-      link="base_link" />
+      link="base_link_arm" />
     <child
       link="Link1" />
@@ -139,6 +162,6 @@
       xyz="0 -1 0" />
     <limit
-      lower="-3.5"
-      upper="3.5"
+      lower="-3.1"
+      upper="3.1"
       effort="60"
       velocity="3.14" />
@@ -200,6 +223,6 @@
       xyz="0 1 0" />
     <limit
-      lower="-3.5"
-      upper="3.5"
+      lower="-2.268"
+      upper="2.268"
       effort="60"
       velocity="3.14" />
@@ -261,6 +284,6 @@
       xyz="0 -1 0" />
     <limit
-      lower="-3.5"
-      upper="3.5"
+      lower="-3.1"
+      upper="3.1"
       effort="30"
       velocity="3.92" />
@@ -322,6 +345,6 @@
       xyz="0 1 0" />
     <limit
-      lower="-3.5"
-      upper="3.5"
+      lower="-2.355"
+      upper="2.355"
       effort="30"
       velocity="3.92" />
@@ -383,6 +406,6 @@
       xyz="0 -1 0" />
     <limit
-      lower="-3.5"
-      upper="3.5"
+      lower="-3.1"
+      upper="3.1"
       effort="10"
       velocity="3.92" />
@@ -444,6 +467,6 @@
       xyz="0 1 0" />
     <limit
-      lower="-3.5"
-      upper="3.5"
+      lower="-2.233"
+      upper="2.233"
       effort="10"
       velocity="3.92" />
@@ -541,3 +564,7 @@
     </plugin>
   </gazebo>
+  <!-- kinectdk -->  <!-- ${-M_PI/2} -->
+  <xacro:property name="M_PI" value="3.1415926535897931" />
+	<xacro:include filename="$(find fabo_arm7_gazebo)/urdf/kinectdk.urdf.xacro"/>
+	<xacro:sensor_kinectdk parent="Link7"  cam_oy="0"   dis_py_between_rgb_and_depth="0.0"/>
 </robot>

File: rm_75_description/urdf/rm_75_bottom【此文件是原版。目前使用的_bottom是扩大关节活动范围的】.urdf.xacro (robot description, xacro)
@@ -139,6 +139,6 @@
       xyz="0 -1 0" />
     <limit
-      lower="-3.5"
-      upper="3.5"
+      lower="-3.1"
+      upper="3.1"
       effort="60"
       velocity="3.14" />
@@ -200,6 +200,6 @@
       xyz="0 1 0" />
     <limit
-      lower="-3.5"
-      upper="3.5"
+      lower="-2.268"
+      upper="2.268"
       effort="60"
       velocity="3.14" />
@@ -261,6 +261,6 @@
       xyz="0 -1 0" />
     <limit
-      lower="-3.5"
-      upper="3.5"
+      lower="-3.1"
+      upper="3.1"
       effort="30"
       velocity="3.92" />
@@ -322,6 +322,6 @@
       xyz="0 1 0" />
     <limit
-      lower="-3.5"
-      upper="3.5"
+      lower="-2.355"
+      upper="2.355"
       effort="30"
       velocity="3.92" />
@@ -383,6 +383,6 @@
       xyz="0 -1 0" />
     <limit
-      lower="-3.5"
-      upper="3.5"
+      lower="-3.1"
+      upper="3.1"
       effort="10"
       velocity="3.92" />
@@ -444,6 +444,6 @@
       xyz="0 1 0" />
     <limit
-      lower="-3.5"
-      upper="3.5"
+      lower="-2.233"
+      upper="2.233"
       effort="10"
       velocity="3.92" />
